File: CodeName0.kicad_sch (KiCad schematic)
At the start: 44 parts, among them J1 Conn Debug, J2 USB C 16p, J3 Micro_SD_Card_Det1, SW1 Tactile Switch, SW2 Tactile Switch, U1 STM32H743VITx, U2 AMS1117-3.3, Y1 Crystal_GND24

Commit message: feat: layouting PCB
Parts:
- removed C13, C14, C15: 10uF, Capacitor_SMD:C_0805_2012Metric, symbol Device:C_Small
- added C10, C24, C32: 10uF, Capacitor_SMD:C_1206_3216Metric, symbol Device:C_Small
- added C2: 470uF, Capacitor_SMD:CP_Elec_10x10.5, symbol Device:C_Small
- added C25, C26, C28, C29, C3, C30, C31, C4, C7: 100nF, Capacitor_SMD:C_0603_1608Metric, symbol Device:C_Small
- added C27: 220nF, Capacitor_SMD:C_0603_1608Metric, symbol Device:C_Small
- added C5, C6, C8: 22uF, Capacitor_SMD:C_1206_3216Metric, symbol Device:C_Small
- added C9: 10nF, Capacitor_SMD:C_0603_1608Metric, symbol Device:C_Small
- added D3: LED, LED_SMD:LED_0805_2012Metric, symbol Device:LED
- added D4, D6: LED, LED_SMD:LED_0603_1608Metric, symbol Device:LED
- added D5: 1N4148WS, Diode_SMD:D_SOD-323, symbol Diode:1N4148WS
- added J2: Power Conn, Connector_JST:JST_GH_SM07B-GHS-TB_1x07-1MP_P1.25mm_Horizontal, symbol Connector:Conn_01x07_Pin
- added J4: Telemetry Conn, Connector_JST:JST_GH_SM04B-GHS-TB_1x04-1MP_P1.25mm_Horizontal, symbol Connector:Conn_01x04_Pin
- added J6: GPS Conn, Connector_JST:JST_GH_SM06B-GHS-TB_1x06-1MP_P1.25mm_Horizontal, symbol Connector:Conn_01x06_Pin
- added J7: Buzzer Conn, Connector_JST:JST_GH_SM02B-GHS-TB_1x02-1MP_P1.25mm_Horizontal, symbol Connector:Conn_01x02_Pin
- added J8: ESP32 Jumper Conn, Connector_PinHeader_2.54mm:PinHeader_2x03_P2.54mm_Vertical, symbol Connector_Generic:Conn_02x03_Odd_Even
- added J9: ESP32 Programming Conn, Connector_PinHeader_2.54mm:PinHeader_1x03_P2.54mm_Vertical, symbol Connector:Conn_01x03_Pin
- added L1: 15uH, Inductor_SMD:L_Sunlord_SWPA6045S, symbol Device:L_Small
- added Q1: MMBT3904, Package_TO_SOT_SMD:SOT-23, symbol Transistor_BJT:MMBT3904
- added R17: 18K, Resistor_SMD:R_0603_1608Metric, symbol Device:R_Small
- added R18, R22: 1K, Resistor_SMD:R_0603_1608Metric, symbol Device:R_Small
- added R2: 100K, Resistor_SMD:R_0603_1608Metric, symbol Device:R_Small
- added R20, R21, R23: 330, Resistor_SMD:R_0603_1608Metric, symbol Device:R_Small
- added R26, R27: 4.7K, Resistor_SMD:R_0603_1608Metric, symbol Device:R_Small
- added R28, R29, R3, R30, R9: 10K, Resistor_SMD:R_0603_1608Metric, symbol Device:R_Small
- added R5: 30.9K, Resistor_SMD:R_0603_1608Metric, symbol Device:R_Small
- added SW3, SW4: Tactile Switch, Button_Switch_SMD:SW_Push_SPST_NO_Alps_SKRK, symbol Switch:SW_Push
- added U1: TPS5430DDAR, TPS5430DDAR:CONV_TPS5430DDAR, symbol TPS5430DDAR:TPS5430DDAR
- added U4: ICM-42688-P, ICM-42688-P:PQFN50P300X250X97-14N, symbol ICM-42688-P:ICM-42688-P
- added U5: BMP388, BMP388:PQFN50P200X200X80-10N, symbol BMP388:BMP388
- added U6: ESP32 C3 WROOM 02U, RF_Module:ESP32-C3-WROOM-02U, symbol RF_Module:ESP32-C3-WROOM-02U
- C16: value 100nF -> 10uF; footprint Capacitor_SMD:C_0603_1608Metric -> Capacitor_SMD:C_1206_3216Metric
- J1: value Conn Debug -> STM32 Debug Conn
- J5: renamed from J3; value Micro_SD_Card_Det1 -> MicroSD
- U2: value AMS1117-3.3 -> LDO
- renumbered C17 to C1, C1 to C11, C4 to C12, C11 to C13, C12 to C14, C2 to C15, C5 to C17, C3 to C18, C10 to C19, C6 to C20, C7 to C21, C8 to C22, C9 to C23, FB2 to FB1, FB1 to FB2, J2 to J3, R11 to R1, R13 to R10, R5 to R11, R6 to R12, R15 to R13, R9 to R14, R7 to R15, R8 to R16, R10 to R19, R1 to R24, R2 to R25, R12 to R4, R3 to R6, R4 to R7, R14 to R8, U1 to U3
Connections:
- net +3V3 is gone; now on net +3.3V: C16.1, U2.2 (VO)
- net +3.3V: now also U3.20 (VREF+), C24.1, C25.1, C26.1, C27.2, C28.1, C29.2, C30.1, C31.1, C32.2, J4.1 (Pin_1), J6.1 (Pin_1), R21.2, R23.2, R26.1, R27.1, R28.2, R29.2, R30.2, SW3.1, SW4.1, U4.5 (VDDIO), U4.8 (VDD), U5.1 (VDDIO), U5.10 (VDD), U5.6 (CSB), U6.1 (3V3); no longer C20.1, C21.1, FB2.2
- net +5V: now also D1.1 (K), D2.1 (K), U2.3 (VI), C10.1, J7.1 (Pin_1); no longer D1.2 (A)
- net GND: now also C10.2, C2.2, C24.2, C25.2, C26.2, C27.1, C28.2, C29.1, C3.2, C30.2, C31.2, C32.1, C4.2, C5.2, C6.2, C7.2, C8.2, D3.1 (K), D4.1 (K), D6.1 (K), J2.2 (Pin_2), J4.4 (Pin_4), J6.6 (Pin_6), J9.3 (Pin_3), Q1.2 (E), R18.1, R3.1, R9.1, SW3.2, SW4.2, U1.6 (GND), U1.9 (POWERPAD), U4.10 (RESV_10), U4.11 (RESV_11), U4.2 (RESV_2), U4.3 (RESV_3), U4.6 (GND), U4.7 (RESV_7), U4.9 (INT2/FSYNC/CLKIN), U5.3 (VSS), U5.5 (SDO), U5.8 (VSS), U5.9 (VSS), U6.19 (GND), U6.9 (GND)
- net at R14.2: now also D2.2 (A), J3.A4 (VBUS), J3.A9 (VBUS), J3.B4 (VBUS), J3.B9 (VBUS); no longer D2.1 (K)
- net SHIELD: now reaches FB1.1, J3.S1 (SHIELD)
- net ADC_VBATT: now reaches U3.22 (PA0)
- net ADC_VBATT: now also C7.1, R17.2, R18.2
- net ADC_CURR: now reaches U3.23 (PA1)
- net ADC_CURR: now also J2.3 (Pin_3), R9.2
- net USART2_TX: now reaches U3.24 (PA2)
- net USART2_TX: now also J8.1 (Pin_1)
- net USART2_RX: now reaches U3.25 (PA3)
- net USART2_RX: now also J8.2 (Pin_2)
- net GPIO_EXTI4: now reaches U3.28 (PA4)
- net GPIO_EXTI4: now also U4.4 (INT1/INT)
- net SPI1_SCK: now reaches U3.29 (PA5)
- net SPI1_SCK: now also U4.13 (AP_SCL/AP_SCLK)
- net SPI1_MISO: now reaches U3.30 (PA6)
- net SPI1_MISO: now also U4.1 (AP_SDO/AP_AD0)
- net SPI1_MOSI: now reaches U3.31 (PA7)
- net SPI1_MOSI: now also U4.14 (AP_SDA/AP_SDIO/AP_SDI)
- net TIM_CH1: now reaches U3.39 (PE9)
- net TIM_CH1: now also J2.4 (Pin_4)
- net TIM_CH2: now reaches U3.41 (PE11)
- net TIM_CH2: now also J2.5 (Pin_5)
- net TIM_CH3: now reaches U3.43 (PE13)
- net TIM_CH3: now also J2.6 (Pin_6)
- net TIM_CH4: now reaches U3.44 (PE14)
- net TIM_CH4: now also J2.7 (Pin_7)
- net USART3_TX: now reaches U3.46 (PB10)
- net USART3_TX: now also J4.3 (Pin_3)
- net USART3_RX: now reaches U3.47 (PB11)
- net USART3_RX: now also J4.2 (Pin_2)
- net GPIO_SPI_CS: now reaches U3.67 (PA8)
- net GPIO_SPI_CS: now also R28.1, U4.12 (AP_CS)
- net GPIO_BUZZER: now reaches U3.69 (PA10)
- net GPIO_BUZZER: now also R22.1
- net GPIO_LED: now reaches U3.7 (PC13)
- net GPIO_LED: now also R20.2
- net GPIO_EXTI14: now reaches U3.8 (PC14)
- net GPIO_EXTI14: now also U5.7 (INT)
- net USART1_TX: now reaches U3.92 (PB6)
- net USART1_TX: now also J6.3 (Pin_3)
- net USART1_RX: now reaches U3.93 (PB7)
- net USART1_RX: now also J6.2 (Pin_2)
- net I2C1_SCL: now reaches U3.95 (PB8)
- net I2C1_SCL: now also J6.4 (Pin_4), R26.2, U5.2 (SCK)
- net I2C1_SDA: now reaches U3.96 (PB9)
- net I2C1_SDA: now also J6.5 (Pin_5), R27.2, U5.4 (SDI)
- new net: R3.2, R5.2, U1.4 (VSENSE)
- new net: C20.1, C21.1, FB2.2
- new net: C4.1, C5.1, C6.1, C8.1, D1.2 (A), L1.2, R5.1
- new net: R29.1, U6.2 (EN)
- new net: D3.2 (A), R20.1
- new net: C9.1, U1.1 (BOOT)
- new net: C9.2, L1.1, U1.8 (PH)
- new net: D6.2 (A), R23.1
- new net: D4.2 (A), R21.1
- new net: R2.1, U1.5 (ENA)
- new net: D5.1 (K), J7.2 (Pin_2)
- new net: Q1.1 (B), R22.2
- new net: D5.2 (A), Q1.3 (C)
- new net: R30.1, U6.8 (IO9)
- new net +BATT: C2.1, C3.1, J2.1 (Pin_1), R17.1, R2.2, U1.7 (VIN)
- new net ESP32_RX: J8.3 (Pin_3), U6.11 (IO20/RXD)
- new net ESP32_TX: J8.4 (Pin_4), U6.12 (IO21/TXD)
- new net ESP_PROG_RX: J8.6 (Pin_6), J9.1 (Pin_1)
- new net ESP_PROG_TX: J8.5 (Pin_5), J9.2 (Pin_2)
- no-connect marks 3 -> 62
Other:
- note added: "BMP388 Module"
- note added: "Buck Converter"
- note added: "Connectors"
- note added: "ESP32 C3 Module"
- note added: "ICM-42688-P 6DOF IMU Sensor"
- note added: "MicroSD"
- note added: "USB Conenctor"
- note added: "VDD and VDDA Decoupling"
- note added: "Voltage Regulator"
- note removed: "Debug Connector"
- note removed: "Power Supply"
- note removed: "USB C Connector"
- note removed: "VDD & VDDA Decoupling"
- moved on the sheet: C1, C11, C12, C13, C14, C15, C17, C18, C19, C20, C21, C22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

Commit message: feat: remove esp32-c3 wroom
Parts:
- removed C24: 10uF, Capacitor_SMD:C_1206_3216Metric, symbol Device:C_Small
- removed C25, C26, C28: 100nF, Capacitor_SMD:C_0603_1608Metric, symbol Device:C_Small
- removed D4: LED, LED_SMD:LED_0603_1608Metric, symbol Device:LED
- removed J1: STM32 Debug Conn, Connector_PinHeader_2.54mm:PinHeader_1x03_P2.54mm_Vertical, symbol Connector:Conn_01x03_Pin
- removed J8: ESP32 Jumper Conn, Connector_PinHeader_2.54mm:PinHeader_2x03_P2.54mm_Vertical, symbol Connector_Generic:Conn_02x03_Odd_Even
- removed J9: ESP32 Programming Conn, Connector_PinHeader_2.54mm:PinHeader_1x03_P2.54mm_Vertical, symbol Connector:Conn_01x03_Pin
- removed R21: 330, Resistor_SMD:R_0603_1608Metric, symbol Device:R_Small
- removed R29, R30: 10K, Resistor_SMD:R_0603_1608Metric, symbol Device:R_Small
- removed SW3, SW4: Tactile Switch, Button_Switch_SMD:SW_Push_SPST_NO_Alps_SKRK, symbol Switch:SW_Push
- removed U6: ESP32 C3 WROOM 02U, RF_Module:ESP32-C3-WROOM-02U, symbol RF_Module:ESP32-C3-WROOM-02U
- added J1: STM32 Debug Conn, Connector_PinHeader_2.54mm:PinHeader_1x04_P2.54mm_Vertical, symbol Connector:Conn_01x04_Pin
Connections:
- net +3.3V: now also J1.1 (Pin_1)
- net GND: now also J1.4 (Pin_4)
- net SWCLK: now also J1.3 (Pin_3)
- net SWDIO: now also J1.2 (Pin_2)
- net TIM3_CH3: now reaches U3.34 (PB0)
- net TIM3_CH4: now reaches U3.35 (PB1)
- net UART4_RX: now reaches U3.81 (PD0)
- net UART4_TX: now reaches U3.82 (PD1)
- net TIM3_CH1: now reaches U3.90 (PB4)
- net TIM3_CH2: now reaches U3.91 (PB5)
- no-connect marks 62 -> 44
Other:
- note removed: "ESP32 C3 Module"
- moved on the sheet: C17, C20, C21, C22, C23, C27, C29, C30, C31, C32, D6, FB2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

Commit message: feat: ESP32-C3 schematic and pcb layout
Parts:
- removed J1: STM32 Debug Conn, Connector_PinHeader_2.54mm:PinHeader_1x04_P2.54mm_Vertical, symbol Connector:Conn_01x04_Pin
- added C24, C25, C36: 1uF, Capacitor_SMD:C_0805_2012Metric, symbol Device:C_Small
- added C26: 10nF, Capacitor_SMD:C_0603_1608Metric, symbol Device:C_Small
- added C28, C34, C35, C37, C39: 100nF, Capacitor_SMD:C_0603_1608Metric, symbol Device:C_Small
- added C33: 10uF, Capacitor_SMD:C_0805_2012Metric, symbol Device:C_Small
- added C38: 1pF, Capacitor_SMD:C_0402_1005Metric, symbol Device:C_Small
- added C40, C41: 15pF, Capacitor_SMD:C_0603_1608Metric, symbol Device:C_Small
- added C42: 1.5pF, Capacitor_SMD:C_0402_1005Metric, symbol Device:C_Small
- added C43: 100pF, Capacitor_SMD:C_0402_1005Metric, symbol Device:C_Small
- added D4: LED, LED_SMD:LED_0805_2012Metric, symbol Device:LED
- added D7: LED, LED_SMD:LED_0603_1608Metric, symbol Device:LED
- added D8: SS34, Diode_SMD:D_SMA, symbol Diode:SS34
- added FB3: FerriteBead, Inductor_SMD:L_0603_1608Metric, symbol Device:FerriteBead_Small
- added J1: STM32 Debug Conn, Connector_PinHeader_2.54mm:PinHeader_1x03_P2.54mm_Vertical, symbol Connector:Conn_01x03_Pin
- added J10: Telemetry 2 Conn, Connector_JST:JST_GH_SM04B-GHS-TB_1x04-1MP_P1.25mm_Horizontal, symbol Connector:Conn_01x04_Pin
- added J11: I2C, Connector_JST:JST_GH_BM04B-GHS-TBT_1x04-1MP_P1.25mm_Vertical, symbol Connector:Conn_01x04_Pin
- added J12: PWM Aux Conn, Connector_PinHeader_2.54mm:PinHeader_2x03_P2.54mm_Vertical, symbol Connector_Generic:Conn_02x03_Top_Bottom
- added J8: U.FL Hirose, Connector_Coaxial:U.FL_Hirose_U.FL-R-SMT-1_Vertical, symbol Connector:Conn_Coaxial
- added J9: ESP32 Prog Conn, Connector_PinHeader_2.54mm:PinHeader_1x04_P2.54mm_Vertical, symbol Connector:Conn_01x04_Pin
- added L2: 1.8nH, Inductor_SMD:L_0402_1005Metric, symbol Device:L_Small
- added R21, R29, R30, R31: 10K, Resistor_SMD:R_0603_1608Metric, symbol Device:R_Small
- added R32, R33: 330, Resistor_SMD:R_0603_1608Metric, symbol Device:R_Small
- added SW3, SW4: Tactile Switch, Button_Switch_SMD:SW_Push_SPST_NO_Alps_SKRK, symbol Switch:SW_Push
- added U6: ESP32-C3FH4, ESP32-C3FH4:QFN50P500X500X90-33N, symbol ESP32-C3FH4:ESP32-C3FH4
- added U7: BCT4222CEAB-TR, Package_SO:MSOP-10_3x3mm_P0.5mm, symbol BCT4222CEAB-TR:BCT4222CEAB-TR
- added Y2: Crystal 40MHz, Crystal:Crystal_SMD_3225-4Pin_3.2x2.5mm, symbol Device:Crystal_GND24
- J4: value Telemetry Conn -> Telemetry 1 Conn
- R26, R27: value 4.7K -> 2.2K
- U2: value LDO -> AMS1117-3.3
- Y1: value Crystal_GND24 -> Crystal 25Mhz
Connections:
- net +3.3V: now also C24.2, C25.1, C26.2, C28.1, C33.1, C34.1, C35.1, C36.1, C39.2, D8.2 (A), FB3.1, J10.1 (Pin_1), J11.1 (Pin_1), R21.1, R29.1, R33.2, U6.11 (VDD3P3_RTC), U6.17 (VDD3P3_CPU), U6.18 (VDD_SPI), U6.2 (VDD3P3), U6.3 (VDD3P3), U6.31 (VDDA), U6.32 (VDDA), U7.10 (VCC)
- net GND: now also C24.1, C25.2, C26.1, C28.2, C33.2, C34.2, C35.2, C36.2, C37.1, C39.1, C40.2, C41.2, C42.1, D4.1 (K), D7.1 (K), FB3.2, J1.3 (Pin_3), J10.4 (Pin_4), J11.4 (Pin_4), J12.5 (Pin_5), J8.2 (Ext), J9.4 (Pin_4), R31.1, SW3.1, SW4.1, U6.33 (GND), U7.5 (GND), U7.9 (OE), Y2.2, Y2.4
- net I2C1_SCL: now also J11.2 (Pin_2)
- net I2C1_SDA: now also J11.3 (Pin_3)
- net SWCLK: now also J1.2 (Pin_2)
- net SWDIO: now also J1.1 (Pin_1)
- net TIM3_CH1: now also J12.1 (Pin_1)
- net TIM3_CH2: now also J12.2 (Pin_2)
- net TIM3_CH3: now also J12.3 (Pin_3)
- net TIM3_CH4: now also J12.4 (Pin_4)
- net UART4_RX: now also J10.2 (Pin_2)
- net UART4_TX: now also J10.3 (Pin_3)
- net USART2_RX: now also U7.8 (HSD1-)
- net USART2_TX: now also U7.2 (HSD1+)
- new net: D7.2 (A), R33.1
- new net: C38.1, C42.2, L2.1
- new net: C43.1, L2.2
- new net: R30.2, R31.2, U7.1 (S)
- new net: D4.2 (A), R32.1
- new net: C38.2, J8.1 (In)
- new net: D8.1 (K), J12.6 (Pin_6)
- new net ESP32_BOOT: R29.2, SW3.2, U6.15 (GPIO9)
- new net ESP32_EN: C37.2, R21.2, SW4.2, U6.7 (CHIP_EN)
- new net ESP32_LNA_IN: C43.2, U6.1 (LNA_IN)
- new net ESP32_MISO: U6.6 (GPIO2)
- new net ESP32_MOSI: U6.13 (GPIO7/MTDO)
- new net ESP32_NSS: U6.8 (GPIO3)
- new net ESP32_PROG_RX: J9.2 (Pin_2), U7.7 (HSD2-)
- new net ESP32_PROG_TX: J9.3 (Pin_3), U7.3 (HSD2+)
- new net ESP32_RX: U6.27 (GPIO20/U0RXD), U7.4 (D+)
- new net ESP32_SCK: U6.12 (GPIO6/MTCK)
- new net ESP32_STATUS_LED: R32.2, U6.10 (GPIO5/MTDI)
- new net ESP32_TX: U6.28 (GPIO21/U0TXD), U7.6 (D-)
- new net SX_BUSY: U6.16 (GPIO10)
- new net SX_DIO1: U6.14 (GPIO8)
- new net SX_RESET: U6.9 (GPIO4/MTMS)
- new net USB_UART_3V3: J9.1 (Pin_1), R30.1
- new net XTAL_N: C41.1, U6.29 (XTAL_N), Y2.3
- new net XTAL_P: C40.1, U6.30 (XTAL_P), Y2.1
- no-connect marks 44 -> 54
Other:
- note added: "BMP388 Barometric Sensor"
- note added: "ESP32 Analog Switch"
- note added: "ESP32 Antenna"
- note added: "ESP32 BOOT & RESET"
- note added: "ESP32 Connectors"
- note added: "ESP32 Crystal"
- note added: "ESP32 LED"
- note added: "ESP32-C3H4"
- note added: "STM32 BOOT0 & NSRT"
- note added: "STM32 Connectors"
- note added: "STM32 Crystal"
- note added: "STM32 LED"
- note added: "STM32 MicroSD"
- note added: "STM32 USB Conenctor"
- note added: "STM32 VDD and VDDA Decoupling"
- note removed: "BMP388 Module"
- note removed: "BOOT0 & NSRT"
- note removed: "Connectors"
- note removed: "Crystal"
- note removed: "MicroSD"
- note removed: "USB Conenctor"
- note removed: "VDD and VDDA Decoupling"
- moved on the sheet: C13, C14, C19, C22, C23, C27, C29, C32, D3, D5, D6, J7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

Commit message: feat: SX1280
Parts:
- added C44: 470nF, Capacitor_SMD:C_0603_1608Metric, symbol Device:C_Small
- added C45: 10nF, Capacitor_SMD:C_0603_1608Metric, symbol Device:C_Small
- added C46, C48, C49: 100nF, Capacitor_SMD:C_0603_1608Metric, symbol Device:C_Small
- added C47: 10uF, Capacitor_SMD:C_1206_3216Metric, symbol Device:C_Small
- added C50: 1nF, Capacitor_SMD:C_0603_1608Metric, symbol Device:C_Small
- added FB4, FB5, FB6, FB7: FerriteBead, Inductor_SMD:L_0603_1608Metric, symbol Device:FerriteBead_Small
- added L3: 15uH, Inductor_SMD:L_Changjiang_FNR3015S, symbol Device:L_Small
- added R34: 10K, Resistor_SMD:R_0603_1608Metric, symbol Device:R_Small
- added U8: SX1280IMLTRT, SX1280IMLTRT:XCVR_SX1280IMLTRT, symbol SX1280IMLTRT:SX1280IMLTRT
- added Y3: OW7EL89CENUNFAYLC-52M, Crystal:Crystal_SMD_2016-4Pin_2.0x1.6mm, symbol Device:Crystal_GND24
- C24: value 1uF -> 10nF; footprint Capacitor_SMD:C_0805_2012Metric -> Capacitor_SMD:C_0603_1608Metric
- C25: value 1uF -> 100nF; footprint Capacitor_SMD:C_0805_2012Metric -> Capacitor_SMD:C_0603_1608Metric
- C26: value 10nF -> 1uF; footprint Capacitor_SMD:C_0603_1608Metric -> Capacitor_SMD:C_0805_2012Metric
- C33: value 10uF -> 1uF
- C34: value 100nF -> 1uF; footprint Capacitor_SMD:C_0603_1608Metric -> Capacitor_SMD:C_0805_2012Metric
- C36: value 1uF -> 10uF; footprint Capacitor_SMD:C_0805_2012Metric -> Capacitor_SMD:C_1206_3216Metric
- L1: footprint Inductor_SMD:L_Sunlord_SWPA6045S -> Inductor_SMD:L_Changjiang_FNR4020S
- Y1: value Crystal 25Mhz -> X322525MOB4SI
- Y2: value Crystal 40MHz -> X322540MPB4SI
Connections:
- net +3.3V: now also C24.1, C26.1, C46.1, C47.1, C48.2, C49.1, FB4.1, FB5.1, FB6.1, FB7.1, U8.1 (VR_PA), U8.11 (VBAT_IO), U8.15 (VBAT), Y3.4; no longer C24.2, C26.2
- net ESP32_MISO: now also U8.16 (MISO_TX)
- net ESP32_MOSI: now also U8.17 (MOSI_RX)
- net ESP32_NSS: now also U8.19 (~{SS_CTS})
- net ESP32_SCK: now also U8.18 (SCK_~{RTS})
- net GND: now also C24.2, C26.2, C44.2, C45.1, C46.2, C47.2, C48.1, C49.2, FB4.2, FB5.2, FB6.2, FB7.2, R34.2, U8.13 (GND), U8.20 (GND), U8.21 (GND), U8.23 (GND), U8.24 (GND), U8.5 (GND), Y3.1, Y3.2; no longer C24.1, C26.1
- net SX_BUSY: now also U8.7 (BUSY)
- net SX_DIO1: now also U8.8 (DIO1)
- net SX_RESET: now also U8.3 (~{RESET})
- new net: C44.1, C45.2, L3.1, U8.12 (DCC_FB), U8.2 (VDD_IN)
- new net: L3.2, U8.14 (DCC_SW)
- new net: C50.2, R34.1, Y3.3
- new net SX_XTA: C50.1, U8.4 (XTA)
- no-connect marks 54 -> 57
Other:
- note added: "SX1280 & TCXO Crystal"
- moved on the sheet: C22, C23, C27, C29, C32, C37, C38, C39, C40, C41, C42, C43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

Commit message: feat: redesign power archtecture and integrate SX1280
Parts:
- removed D1: SS34, Diode_SMD:D_SMA, symbol Diode:SS34
- added C51: 100nF, Capacitor_SMD:C_0603_1608Metric, symbol Device:C_Small
- added C52: 47pF, Capacitor_SMD:C_0402_1005Metric, symbol Device:C_Small
- added C53: 1nF, Capacitor_SMD:C_0603_1608Metric, symbol Device:C_Small
- added C54, C55: 100uF, Capacitor_SMD:C_1206_3216Metric, symbol Device:C_Small
- added D1: SMBJ15A, Diode_SMD:D_SMB, symbol Diode:SM6T15A
- added D10, D11: DSK34, Diode_SMD:D_SOD-123F, symbol Diode:SS34
- added D9: SS34, Diode_SMD:D_SMA, symbol Diode:SS34
- added FL1: 2450FM07D0034T, 2450FM07D0034T:FIL_2450FM07D0034T, symbol 2450FM07D0034T:2450FM07D0034T
- added J13: U.FL Hirose, Connector_Coaxial:U.FL_Hirose_U.FL-R-SMT-1_Vertical, symbol Connector:Conn_Coaxial
- added L4: 6.8uH, Inductor_SMD:L_Sunlord_MWSA0503S, symbol Device:L_Small
- added Q2: AO3401A, Package_TO_SOT_SMD:SOT-23, symbol Transistor_FET:AO3401A
- added R35: 3.3K, Resistor_SMD:R_0603_1608Metric, symbol Device:R_Small
- added R36: 332K, Resistor_SMD:R_0603_1608Metric, symbol Device:R_Small
- added R37: 10K, Resistor_SMD:R_0603_1608Metric, symbol Device:R_Small
- added R38: 30K, Resistor_SMD:R_0603_1608Metric, symbol Device:R_Small
- added U9: TPS54331DR, TPS54331DR:SOIC127P599X175-8N, symbol TPS54331DR:TPS54331DR
- C2: value 470uF -> 22uF; footprint Capacitor_SMD:CP_Elec_10x10.5 -> Capacitor_SMD:C_1206_3216Metric
- C6: value 22uF -> 100uF
- C8: value 22uF -> 100nF; footprint Capacitor_SMD:C_1206_3216Metric -> Capacitor_SMD:C_0603_1608Metric
- C9: value 10nF -> 100nF
- L1: footprint Inductor_SMD:L_Changjiang_FNR4020S -> Inductor_SMD:L_Bourns_SRP7028A_7.3x6.6mm
- R3: value 10K -> 3.3K
- R5: value 30.9K -> 10K
Connections:
- net +3.3V: now also D10.1 (K), D11.1 (K); no longer C16.1, U2.2 (VO)
- net +5V: now also C4.1, C6.1, J3.A4 (VBUS), J3.A9 (VBUS), J3.B4 (VBUS), J3.B9 (VBUS), L1.1, R14.2, R5.1, C54.1; no longer D2.1 (K)
- net +BATT: now also C5.1, D1.1 (A1), Q2.2 (S), Q2.3 (D), R36.2, U9.2 (VIN)
- net GND: now also D2.2 (A), U8.25 (EXP), C52.2, C54.2, C55.1, D1.2 (A2), D9.2 (A), FL1.2, FL1.4, J13.2 (Ext), Q2.1 (G), R35.1, R38.2, U9.7 (GND)
- net SX_RFIO: now reaches U8.22 (RFIO)
- net SX_RFIO: now also FL1.1
- net at C9.2, U1.8 (PH): now also D2.1 (K), L1.2; no longer L1.1
- new net: C55.2, D11.2 (A), L4.2, R37.1
- new net: C53.1, R38.1
- new net: C52.1, C53.2, U9.6 (COMP)
- new net: C8.1, U9.4 (SS)
- new net: FL1.3, J13.1 (In)
- new net: C51.1, D9.1 (K), L4.1, U9.8 (PH)
- new net: C16.1, D10.2 (A), U2.2 (VO)
- new net: C51.2, U9.1 (BOOT)
- new net: R36.1, U9.3 (EN)
- new net: R35.2, R37.2, U9.5 (VSENSE)
Other:
- note added: "3.3V Buck Converter"
- note added: "5V Buck Converter"
- note added: "ESP32 Antenna Connector"
- note added: "SX1280 Antenna Connector"
- note removed: "Buck Converter"
- note removed: "ESP32 Antenna"
- moved on the sheet: C1, C27, C29, C3, C30, C31, C32, C4, C45, C7, C9, D3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

Commit message: feat: polishing and finishing
Parts:
- removed J12: PWM Aux Conn, Connector_PinHeader_2.54mm:PinHeader_2x03_P2.54mm_Vertical, symbol Connector_Generic:Conn_02x03_Top_Bottom
- added C56: 100uF, Capacitor_SMD:C_1206_3216Metric, symbol Device:C_Small
- added D12: LED, LED_SMD:LED_0603_1608Metric, symbol Device:LED
- added J12: AUX Motor Pin, Library:PinHeader_3x04_P2.54mm_Vertical, symbol Connector:Conn_01x12_Pin
- added R39: 330, Resistor_SMD:R_0603_1608Metric, symbol Device:R_Small
- added TP1, TP3, TP5, TP6, TP7: TestPoint, TestPoint:TestPoint_Pad_D1.5mm, symbol Connector:TestPoint
- added TP4: TestPoint, TestPoint:TestPoint_Pad_D2.5mm, symbol Connector:TestPoint
- D8: value SS34 -> DSK34; footprint Diode_SMD:D_SMA -> Diode_SMD:D_SOD-123F
- R3, R35: value 3.3K -> 2.7K
Connections:
- net +3.3V: now also TP7.1; no longer D8.2 (A)
- net +5V: now also D8.1 (K), C56.2, J12.11 (Pin_11), J12.2 (Pin_2), J12.5 (Pin_5), J12.8 (Pin_8), R39.2, TP5.1; no longer C10.1, J3.A4 (VBUS), J3.A9 (VBUS), J3.B4 (VBUS), J3.B9 (VBUS), R14.2, U2.3 (VI)
- net +BATT: now also TP3.1
- net GND: now also D8.2 (A), C56.1, D12.1 (K), J12.12 (Pin_12), J12.3 (Pin_3), J12.6 (Pin_6), J12.9 (Pin_9), TP4.1
- net TIM3_CH1: now also J12.1 (Pin_1)
- net TIM3_CH2: now also J12.4 (Pin_4)
- net TIM3_CH3: now also J12.7 (Pin_7)
- net TIM3_CH4: now also J12.10 (Pin_10)
- net at C55.2, D11.2 (A), L4.2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: now also TP1.1
- new net: D12.2 (A), R39.1
- new net +5V_USB: C10.1, J3.A4 (VBUS), J3.A9 (VBUS), J3.B4 (VBUS), J3.B9 (VBUS), R14.2, TP6.1, U2.3 (VI)
Other:
- moved on the sheet: C10, C16, D1, D10, FL1, J13, Q2, U2
